File: Power.kicad_sch (KiCad schematic)
At the start: 7 parts, among them U1 AMS1117-3.3

Commit message: Add Some Comments
Other:
- note added: "Input: 5V Output: 3V3 1A"
- note added: "Voltage Regulator"
Changed lines of the file:
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@@
 	(generator_version "9.0")
 	(paper "A4")
+	(text "Voltage Regulator"
+		(exclude_from_sim no)
+		(at 127.254 93.98 0)
+		(effects
+			(font
+				(size 2.54 2.54)
+			)
+		)
+	)
+	(text "Input: 5V\nOutput: 3V3 1A"
+		(exclude_from_sim no)
+		(at 119.634 64.262 0)
+		(effects
+			(font
+				(size 1.27 1.27)
+			)
+			(justify left)
+		)
+	)
 	(junction
 		(at 151.13 74.93)
