File: dev_board_STM32H7.kicad_sch (KiCad schematic)
At the start: 13 parts, among them J1 USB_C_Receptacle_USB2.0_16P, J4 Conn_01x05_Pin, J5 Conn_01x04, J6 Conn_01x08

Commit message: Generate output files
Parts:
- added C1, C4: 10uF, Capacitor_SMD:C_0805_2012Metric, symbol Device:C
- added C2, C3: 100nF, Capacitor_SMD:C_0402_1005Metric, symbol Device:C
- added D1: LED, LED_SMD:LED_0603_1608Metric, symbol Device:LED
- added R1: 1k, Resistor_SMD:R_0402_1005Metric, symbol Device:R
- added U1: AMS1117-3.3, Package_TO_SOT_SMD:SOT-223-3_TabPin2, symbol Regulator_Linear:AMS1117-3.3
Connections:
- net +3V3: now also C3.1, C4.1, R1.1, U1.2 (VO)
- net +5V: now also C1.1, C2.1, U1.3 (VI)
- net GND: now also C1.2, C2.2, C3.2, C4.2, D1.1 (K), U1.1 (GND)
- new net: D1.2 (A), R1.2
Other:
- removed sheet Power
- note added: "Input: 5V Output: 3V3 1A"
- note added: "Power Supply"
- moved on the sheet: C20, C5, D3, J1, J4, J5, J6, R2, R3
